Commit message: Added 2nd joint, robot still not fixed..

File: src/cherry_bot_description/urdf/model.urdf (robot description, URDF)
Before this commit: robot cherry_bot, 1 links, 0 joints
Links:
- added link link_1, mass 10; collision cylinder length=0.6 radius=0.2; visual cylinder length=0.6 radius=0.2
- added link link_2, mass 10; collision cylinder length=0.6 radius=0.2; visual cylinder length=0.6 radius=0.2
- added link link_3, mass 10; collision cylinder length=0.6 radius=0.2; visual cylinder length=0.6 radius=0.2
- link base_link: mass 10 -> None; geometry 
Joints:
- added joint J1: type revolute, parent link_1, child link_2, origin xyz=0 0 0.3, axis 1 0 0, limit lower=-1.570 upper=1.570 effort=1000.0 velocity=0.5
- added joint J2: type revolute, parent link_2, child link_3, origin xyz=0 0 0.6, axis 1 0 0, limit lower=-1.570 upper=1.570 effort=1000.0 velocity=0.5
- added joint dummy_joint: type fixed, parent base_link, child link_1

Commit message: changed launch file to start Gazebo in a different way

File: src/cherry_bot_description/urdf/model.urdf (robot description, URDF)
Before this commit: robot cherry_bot, 4 links, 3 joints
Links:
- removed link base_link
- removed link link_3
- added link base
- added link link_0, mass 10; collision cylinder length=0.6 radius=0.2; visual cylinder length=0.6 radius=0.2
Joints:
- removed joint J1
- removed joint J2
- removed joint dummy_joint
- added joint fixed: type fixed, parent base, child link_0
- added joint joint1: type revolute, parent link_0, child link_1, origin xyz=0 0 0.3, axis 1 0 0, limit lower=-1.570 upper=1.570 effort=30.0 velocity=0.5
- added joint joint2: type revolute, parent link_1, child link_2, origin xyz=0 0 0.6, axis 1 0 0, limit lower=-1.570 upper=1.570 effort=30.0 velocity=0.5

Commit message: further adjustments, fixed joint still not fixed...

File: src/cherry_bot_description/urdf/model.urdf (robot description, URDF)
Before this commit: robot cherry_bot, 4 links, 3 joints
Links:
- removed link link_1
- removed link link_2
Joints:
- removed joint fixed
- removed joint joint1
- removed joint joint2
- added joint fixy: type fixed, parent base, child link_0

Commit message: Fixed the robot not attaching to the world frame.

File: src/cherry_bot_description/urdf/model.urdf (robot description, URDF)
Before this commit: robot cherry_bot, 2 links, 1 joints
Links:
- removed link base
- added link link_1, mass 10; collision cylinder length=0.6 radius=0.2; visual cylinder length=0.6 radius=0.2
- added link world
Joints:
- removed joint fixy
- added joint fixed: type fixed, parent world, child link_0
- added joint joint1: type revolute, parent link_0, child link_1, origin xyz=0 0 0.8, axis 1 0 0, limit lower=-1.570 upper=1.570 effort=10000.0 velocity=0.5
